Commit message: fixed the controller_manager  issues

File: src/bumper_bot_description/urdf/bumperbot.urdf.xacro (robot description, xacro)
@@ -4,6 +4,8 @@
     <!-- Include Gazebo Parameters-->
     <xacro:include filename="$(find bumper_bot_description)/urdf/bumperbot_gazebo.xacro"/>
+    <xacro:bumperbot_gazebo is_ignition="$(arg is_ignition)" />
     <!-- Ros2 control-->
     <xacro:include filename="$(find bumper_bot_description)/urdf/bumperbot_ros2_control.xacro"/>
+    <xacro:bumperbot_ros2_control is_ignition="$(arg is_ignition)" />
     <link name="base_footprint"/>
     <link name="base_link">

File: src/bumper_bot_description/urdf/bumperbot_gazebo.xacro (robot description, xacro)
@@ -1,53 +1,46 @@
 <?xml version="1.0"?>
-<robot name="bumperbot" xmlns:xacro="http://www.ros.org/wiki/xacro">
-    <gazebo reference = "wheel_right_link">
-        <mu1>100000000000000.0</mu1>
-        <mu2>100000000000000.0</mu2>
-        <kp>100000000000000.0</kp>
-        <kd>10.0</kd>
-        <minDepth>0.001</minDepth>
-        <maxVel>0.1</maxVel>
-        <fdir>1 0 0</fdir>
-    </gazebo>
-    <gazebo reference = "wheel_left_link">
-        <mu1>100000000000000.0</mu1>
-        <mu2>100000000000000.0</mu2>
-        <kp>100000000000000.0</kp>
-        <kd>10.0</kd>
-        <minDepth>0.001</minDepth>
-        <maxVel>0.1</maxVel>
-        <fdir>1 0 0</fdir>
-    </gazebo>
-    <gazebo reference = "caster_front_link">
-        <mu1>0.1</mu1>
-        <mu2>0.1</mu2>
-        <kp>1000000.0</kp>
-        <kd>100.0</kd>
-        <minDepth>0.001</minDepth>
-        <maxVel>0.1</maxVel>
-        <fdir>1 0 0</fdir>
-    </gazebo>
-    <gazebo reference = "caster_rear_link">
-        <mu1>0.1</mu1>
-        <mu2>0.1</mu2>
-        <kp>1000000.0</kp>
-        <kd>100.0</kd>
-        <minDepth>0.001</minDepth>
-        <maxVel>0.1</maxVel>
-        <fdir>1 0 0</fdir>
-    </gazebo>
-    <gazebo>
-        <xacro:if value="$(arg is_ignition)">
-            <plugin filename="ign_ros2_control-system" name="ign_ros2_control::IgnitionROS2ControlPlugin">
-                <parameter>$(find bumperbot_controllers)/config/bumperbot_controllers.yaml</parameter>
+<robot xmlns:xacro="http://www.ros.org/wiki/xacro">
+    <xacro:macro name="bumperbot_gazebo" params="is_ignition">
+        <gazebo reference="wheel_right_link">
+            <mu1>100000000000000.0</mu1>
+            <mu2>100000000000000.0</mu2>
+            <kp>100000000000000.0</kp>
+            <kd>10.0</kd>
+            <minDepth>0.001</minDepth>
+            <maxVel>0.1</maxVel>
+            <fdir1>1 0 0</fdir1>
+        </gazebo>
+        <gazebo reference="wheel_left_link">
+            <mu1>100000000000000.0</mu1>
+            <mu2>100000000000000.0</mu2>
+            <kp>100000000000000.0</kp>
+            <kd>10.0</kd>
+            <minDepth>0.001</minDepth>
+            <maxVel>0.1</maxVel>
+            <fdir1>1 0 0</fdir1>
+        </gazebo>
+        <gazebo reference="caster_front_link">
+            <mu1>0.1</mu1>
+            <mu2>0.1</mu2>
+            <kp>1000000.0</kp>
+            <kd>100.0</kd>
+            <minDepth>0.001</minDepth>
+            <maxVel>0.1</maxVel>
+            <fdir1>1 0 0</fdir1>
+        </gazebo>
+        <gazebo reference="caster_rear_link">
+            <mu1>0.1</mu1>
+            <mu2>0.1</mu2>
+            <kp>1000000.0</kp>
+            <kd>100.0</kd>
+            <minDepth>0.001</minDepth>
+            <maxVel>0.1</maxVel>
+            <fdir1>1 0 0</fdir1>
+        </gazebo>
+        <gazebo>
+            <plugin filename="gz_ros2_control-system" name="gz_ros2_control::GazeboSimROS2ControlPlugin">
+                <parameters>$(find bumperbot_controllers)/config/bumperbot_controllers.yaml</parameters>
             </plugin>
-        </xacro:if>
-    </gazebo>
-    <gazebo>
-        <xacro:unless value="$(arg is_ignition)">
-            <plugin filename="gz_ros2_control-system" name="gz_ros2_control::GazeboSimROS2ControlPlugin">
-                <parameter> $(find bumperbot_controllers)/config/bumperbot_controllers.yaml </parameter>
-            </plugin>
-        </xacro:unless>
-    </gazebo>
+        </gazebo>
+    </xacro:macro>
 </robot>

File: src/bumper_bot_description/urdf/bumperbot_ros2_control.xacro (robot description, xacro)
@@ -1,31 +1,26 @@
 <?xml version="1.0"?>
-<robot xmlns:xacro="http://www.ros.org/wiki/xacro" name="bumperbot">
-    <ros2_control name="RobotSystem" type="system">
-        <xacro:if  value="$(arg is_ignition)">
+<robot xmlns:xacro="http://www.ros.org/wiki/xacro">
+    <xacro:macro name="bumperbot_ros2_control" params="is_ignition">
+        <ros2_control name="RobotSystem" type="system">
             <hardware>
-                <plugin> ign_ros2_control/IgnitionSystem </plugin>
+                <plugin>gz_ros2_control/GazeboSimSystem</plugin>
             </hardware>
-        </xacro:if>
-        <xacro:unless  value="$(arg is_ignition)">
-            <hardware>
-                <plugin> gz_ros2_control/GazeboSimSystem </plugin>
-            </hardware>
-        </xacro:unless>
-        <joint name="wheel_right_joint">
-            <command_interface name="velocity">
-                <param  name="min">-1</param>
-                <param  name="max">1</param>
-            </command_interface>
-            <state_interface name = "position"/>
-            <state_interface name = "velocity"/>
-        </joint>
-        <joint name="wheel_left_joint">
-            <command_interface name="velocity">
-                <param  name="min">-1</param>
-                <param  name="max">1</param>
-            </command_interface>
-            <state_interface name = "position"/>
-            <state_interface name = "velocity"/>
-        </joint>
-    </ros2_control>
+            <joint name="wheel_right_joint">
+                <command_interface name="velocity">
+                    <param name="min">-1</param>
+                    <param name="max">1</param>
+                </command_interface>
+                <state_interface name="position"/>
+                <state_interface name="velocity"/>
+            </joint>
+            <joint name="wheel_left_joint">
+                <command_interface name="velocity">
+                    <param name="min">-1</param>
+                    <param name="max">1</param>
+                </command_interface>
+                <state_interface name="position"/>
+                <state_interface name="velocity"/>
+            </joint>
+        </ros2_control>
+    </xacro:macro>
 </robot>

Commit message: Added IMU in URDF

File: src/bumper_bot_description/urdf/bumperbot.urdf.xacro (robot description, xacro)
@@ -114,4 +114,26 @@
         </collision>
     </link>
+    <!-- IMU -->
+    <link name = "imu_link">
+        <inertial>
+            <origin xyz="-0.00552433659106688 0.000168210391520346 0.000514000497342681" rpy="0 0 0" />
+            <mass value="0.000528415362211671" />
+            <inertia ixx="1.46176048428261E-08" ixy="1.40015117949421E-10" ixz="-1.99633872937403E-12"
+               iyy="8.59662482954888E-09" iyz="7.52375112767959E-12"
+               izz="2.30279421279312E-08" />
+        </inertial>
+        <visual>
+            <origin rpy = "0 0 0" xyz = "0 0 0" />
+            <geometry>
+                <mesh filename="package://bumper_bot_description/meshes/imu_link.STL" />
+            </geometry>
+        </visual>
+        <collision>
+            <origin rpy = "0 0 0" xyz = "0 0 0" />
+            <geometry>
+                <mesh filename="package://bumper_bot_description/meshes/imu_link.STL" />
+            </geometry>
+        </collision>
+    </link>
     <joint name = "base_joint" type = "fixed">
         <parent link = "base_footprint"/>
@@ -141,3 +163,9 @@
         <origin rpy="0 0 0" xyz="-0.04755 0 -0.0275"/>
     </joint>
+    <joint name = "imu_joint" type = "fixed" >
+        <origin rpy = "0 0 0" xyz = "0 0 0.07" />
+        <parent link = "base_link" />
+        <child link  = "imu_link" />
+        <axis xyz = "0 0 0" />
+    </joint>
 </robot>

File: src/bumper_bot_description/urdf/bumperbot_gazebo.xacro (robot description, xacro)
@@ -42,4 +42,56 @@
                 <parameters>$(find bumperbot_controllers)/config/bumperbot_controllers.yaml</parameters>
             </plugin>
+            <plugin filename="gz-sim-imu-system" name = "gz::sim::systems::Imu">
+            </plugin>
+        </gazebo>
+        <gazebo reference = "imu_link">
+            <sensor name = "imu" type = "imu" >
+                <always_on>True</always_on>
+                <update_rate>100</update_rate>
+                <topic>imu</topic>
+                <gz_frame_id>imu_link</gz_frame_id>
+                <imu>
+                    <angular_velocity>
+                        <x>
+                            <noise type = "gaussian">
+                                <mean>0.0</mean>
+                                <stddev>2e-4</stddev>
+                            </noise>
+                        </x>
+                        <y>
+                            <noise type = "gaussian">
+                                <mean>0.0</mean>
+                                <stddev>2e-4</stddev>
+                            </noise>
+                        </y>
+                        <z>
+                            <noise type = "gaussian">
+                                <mean>0.0</mean>
+                                <stddev>2e-4</stddev>
+                            </noise>
+                        </z>
+                    </angular_velocity>
+                    <linear_acceleration>
+                        <x>
+                            <noise type = "gaussian">
+                                <mean>0.0</mean>
+                                <stddev>1.7e-2</stddev>
+                            </noise>
+                        </x>
+                        <y>
+                            <noise type = "gaussian">
+                                <mean>0.0</mean>
+                                <stddev>1.7e-2</stddev>
+                            </noise>
+                        </y>
+                        <z>
+                            <noise type = "gaussian">
+                                <mean>0.0</mean>
+                                <stddev>1.7e-2</stddev>
+                            </noise>
+                        </z>
+                    </linear_acceleration>
+                </imu>
+            </sensor>
         </gazebo>
     </xacro:macro>
